Commit message: added new k1 models and k1 base walk

File: resources/K1/K1_locomotion.urdf (robot description, URDF)
Before this commit: robot K1, 23 links, 22 joints
Links:
- link Head_1: mass 0.29729 -> 0.30
- link Head_2: mass 0.61387 -> 0.70
- link Left_Ankle_Cross: mass 0.038836 -> 0.039
- link Left_Arm_1: mass 0.45628 -> 0.50
- link Left_Arm_2: mass 0.084303 -> 0.09
- link Left_Arm_3: mass 0.76208 -> 0.80
- link Left_Hip_Pitch: mass 0.64068 -> 0.69
- link Left_Hip_Roll: mass 0.127825 -> 0.13
- link Left_Hip_Yaw: mass 1.5591 -> 1.65
- link Left_Shank: mass 1.483334 -> 1.50
- link Right_Ankle_Cross: mass 0.038836 -> 0.039
- link Right_Arm_1: mass 0.45669 -> 0.50
- link Right_Arm_2: mass 0.083353 -> 0.09
- link Right_Arm_3: mass 0.76234 -> 0.80
- link Right_Hip_Pitch: mass 0.6413 -> 0.69
- link Right_Hip_Roll: mass 0.127825 -> 0.13
- link Right_Hip_Yaw: mass 1.5592 -> 1.65
- link Right_Shank: mass 1.483338 -> 1.50
- link Trunk: mass 6.3921 -> 6.50; geometry collision box size=0.12 0.18 0.2; collision cylinder length=0.1 radius=0.05
- link left_foot_link: mass 0.38305 -> 0.494; geometry collision mesh filename=meshes/Left_Foot.STL; visual mesh filename=meshes/Left_Foot.STL
- link left_hand_link: mass 0.16796 -> 0.19
- link right_foot_link: mass 0.386370 -> 0.494; geometry collision mesh filename=meshes/Right_Foot.STL; visual mesh filename=meshes/Right_Foot.STL
- link right_hand_link: mass 0.16828 -> 0.19
Joints:
- joint AAHead_yaw: limit lower=-1. upper=1. effort=7 velocity=18 -> lower=-1. upper=1. effort=6 velocity=18
- joint ALeft_Shoulder_Pitch: limit lower=-3.316 upper=1.22 effort=10 velocity=18 -> lower=-3.316 upper=1.22 effort=14 velocity=18
- joint ARight_Shoulder_Pitch: limit lower=-3.316 upper=1.22 effort=10 velocity=18 -> lower=-3.316 upper=1.22 effort=14 velocity=18
- joint Head_pitch: limit lower=-0.349 upper=0.855 effort=7 velocity=18 -> lower=-0.349 upper=0.855 effort=6 velocity=18
- joint Left_Ankle_Pitch: limit lower=-0.87 upper=0.345 effort=20 velocity=18 -> lower=-0.87 upper=0.345 effort=20 velocity=18.1
- joint Left_Ankle_Roll: limit lower=-0.345 upper=0.345 effort=15 velocity=18 -> lower=-0.345 upper=0.345 effort=20 velocity=18.1
- joint Left_Elbow_Pitch: limit lower=-2.27 upper=2.27 effort=10 velocity=18 -> lower=-2.27 upper=2.27 effort=14 velocity=18
- joint Left_Elbow_Yaw: limit lower=-2.44 upper=0 effort=10 velocity=18 -> lower=-2.44 upper=0 effort=14 velocity=18
- joint Left_Hip_Pitch: limit lower=-2.21 upper=2.21 effort=30 velocity=18 -> lower=-3.0 upper=2.21 effort=30 velocity=7.1; origin xyz=0 0.096 -0.062 rpy=0 0 0 -> xyz=0 0.096 -0.077 rpy=0 0 0
- joint Left_Hip_Roll: limit lower=-0.4 upper=1.57 effort=20 velocity=18 -> lower=-0.4 upper=1.57 effort=35 velocity=12.9
- joint Left_Hip_Yaw: limit lower=-1. upper=1. effort=20 velocity=18 -> lower=-1. upper=1. effort=20 velocity=18.1
- joint Left_Knee_Pitch: limit lower=0. upper=2.23 effort=40 velocity=18 -> lower=0. upper=2.23 effort=40 velocity=12.5
- joint Left_Shoulder_Roll: limit lower=-1.74 upper=1.57 effort=10 velocity=18 -> lower=-1.74 upper=1.57 effort=14 velocity=18
- joint Right_Ankle_Pitch: limit lower=-0.87 upper=0.345 effort=20 velocity=18 -> lower=-0.87 upper=0.345 effort=20 velocity=18.1
- joint Right_Ankle_Roll: limit lower=-0.345 upper=0.345 effort=15 velocity=18 -> lower=-0.345 upper=0.345 effort=20 velocity=18.1
- joint Right_Elbow_Pitch: limit lower=-2.27 upper=2.27 effort=10 velocity=18 -> lower=-2.27 upper=2.27 effort=14 velocity=18
- joint Right_Elbow_Yaw: limit lower=0 upper=2.44 effort=10 velocity=18 -> lower=0 upper=2.44 effort=14 velocity=18
- joint Right_Hip_Pitch: limit lower=-2.21 upper=2.21 effort=30 velocity=18 -> lower=-3.0 upper=2.21 effort=30 velocity=7.1; origin xyz=0 -0.096 -0.062 rpy=0 0 0 -> xyz=0 -0.096 -0.077 rpy=0 0 0
- joint Right_Hip_Roll: limit lower=-1.57 upper=0.4 effort=20 velocity=18 -> lower=-1.57 upper=0.4 effort=35 velocity=12.9
- joint Right_Hip_Yaw: limit lower=-1. upper=1. effort=20 velocity=18 -> lower=-1. upper=1. effort=20 velocity=18.1
- joint Right_Knee_Pitch: limit lower=0. upper=2.23 effort=40 velocity=18 -> lower=0. upper=2.23 effort=40 velocity=12.5
- joint Right_Shoulder_Roll: limit lower=-1.57 upper=1.74 effort=10 velocity=18 -> lower=-1.57 upper=1.74 effort=14 velocity=18

Commit message: Added KickingK1 import, adjusted BaseWalkK1 parameters, updated YAML configuration for K1, modified URDF for arm orientations, and enhanced entropy loss calculation in runner.

File: resources/K1/K1_locomotion.urdf (robot description, URDF)
Before this commit: robot K1, 23 links, 22 joints
Joints:
- joint Left_Shoulder_Roll: origin xyz=0.0025 0.068 -0.0135 rpy=0 0 0 -> xyz=0.0025 0.068 -0.0135 rpy=-1.35 0 0
- joint Right_Shoulder_Roll: origin xyz=0.0025 -0.068 -0.0135 rpy=0 0 0 -> xyz=0.0025 -0.068 -0.0135 rpy=1.35 0 0
